File: pcb/Ai_Breakout_BME280.sch (EAGLE design)
At the start: 10 parts, among them J1 1X04, J2 1X04NOFIRST, U1 BME280

Commit message: first commit
Parts:
- added U$2: AI-LOGOXS, Ai_Miscellany:AI-LOGOXS
Changed lines of the file:
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@@
 <setting verticaltext="up"/>
 </settings>
-<grid distance="10" unitdist="mil" unit="mil" style="lines" multiple="1" display="yes" altdistance="0.01" altunitdist="inch" altunit="inch"/>
+<grid distance="50" unitdist="mil" unit="mil" style="lines" multiple="1" display="yes" altdistance="0.01" altunitdist="inch" altunit="inch"/>
 <layers>
 <layer number="1" name="Top" color="4" fill="1" visible="no" active="no"/>
@@
 <part name="JS2" library="Ai_Connectors" deviceset="1X02-SJ-NO" device=""/>
 <part name="JS3" library="Ai_Connectors" deviceset="1X02-SJ-NO" device=""/>
+<part name="U$2" library="Ai_Miscellany" deviceset="AI-LOGO" device="XS"/>
 </parts>
 <sheets>
@@
 <instance part="JS2" gate="1" x="149.86" y="116.84" rot="R90"/>
 <instance part="JS3" gate="1" x="105.41" y="116.84" rot="R180"/>
+<instance part="U$2" gate="G$1" x="135.89" y="12.7"/>
 </instances>
 <busses>
