File: pcb/ai_breakout_bme2802.brd (EAGLE design)
At the start: 15.2 x 10.2 mm, 11 parts, among them J1 1X04, J2 1X04NOFIRST, U1 BME280

Commit message: changes and renaming
Parts:
- removed J2: 1X04NOFIRST, Ai_Connectors:1X04-NOFIRST
- removed JS2, JS3: 1X02-SJ-NO, Ai_Connectors:1X02-SJ-NO
- added J3: 1X04, Ai_Connectors:1X04
- added MODE, VDDIO: 1X02-SJ-NO, Ai_Connectors:1X02-SJ-NO
- J1: value 1X04 -> 1X04NOFIRST; device Ai_Connectors:1X04 -> Ai_Connectors:1X04-NOFIRST
- moved U1 0.13 mm to (7.62, 5.08)
- turned J1 to 90 degrees
- renumbered JS1 to PULL-UPS
Connections:
- net CSB: now also J3.2, MODE.1; no longer J2.3, JS2.1
- net GND: now also J1.3, J3.1; no longer J1.2, J2.4
- net SCK: now also J3.4; no longer J2.1
- net SDI: now also J3.3; no longer J2.2
- net SDO: now also J1.1; no longer J1.4
- net VDD: now also J1.4, VDDIO.1; no longer J1.1, JS3.1
- net VDDIO: now also J1.2, MODE.2, VDDIO.2; no longer J1.3, JS2.2, JS3.2
Routing:
- net GND: track 24.0 -> 0.00 mm
Other:
- board text added: "VDDIO"
- board text removed: "IO"
