File: pcb/ai_breakout_bme2802.sch (EAGLE design)
At the start: 11 parts, among them J1 1X04, J2 1X04NOFIRST, U1 BME280

Commit message: changes and renaming
Parts:
- removed J2: 1X04NOFIRST, Ai_Connectors:1X04NOFIRST
- added J3: 1X04, Ai_Connectors:1X04
- J1: value 1X04 -> 1X04NOFIRST; device Ai_Connectors:1X04 -> Ai_Connectors:1X04NOFIRST
- renumbered JS1 to PULL-UPS, JS2 to MODE, JS3 to VDDIO
Connections:
- net CSB: now also J3.2; no longer J2.3
- net GND: now also J1.3, J3.1; no longer J1.2, J2.4
- net SCK: now also J3.4; no longer J2.1
- net SDI: now also J3.3; no longer J2.2
- net SDO: now also J1.1; no longer J1.4
- net VDD: now also J1.4; no longer J1.1
- net VDDIO: now also J1.2; no longer J1.3
Other:
- moved on the sheet: J1
Changed lines of the file:
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@@
 <part name="GND1" library="Ai_Power" deviceset="GND" device=""/>
 <part name="U$1" library="Ai_Power" deviceset="VDD" device=""/>
-<part name="J1" library="Ai_Connectors" deviceset="1X04" device=""/>
-<part name="J2" library="Ai_Connectors" deviceset="1X04" device="NOFIRST" value="1X04NOFIRST"/>
 <part name="GND2" library="Ai_Power" deviceset="GND" device=""/>
 <part name="VDDIO2" library="Ai_Power" deviceset="VDD" device=""/>
-<part name="JS1" library="Ai_Connectors" deviceset="1X02-SJ-NO" device=""/>
-<part name="JS2" library="Ai_Connectors" deviceset="1X02-SJ-NO" device=""/>
-<part name="JS3" library="Ai_Connectors" deviceset="1X02-SJ-NO" device=""/>
+<part name="PULL-UPS" library="Ai_Connectors" deviceset="1X02-SJ-NO" device=""/>
+<part name="MODE" library="Ai_Connectors" deviceset="1X02-SJ-NO" device=""/>
+<part name="VDDIO" library="Ai_Connectors" deviceset="1X02-SJ-NO" device=""/>
 <part name="U$2" library="Ai_Miscellany" deviceset="AI-LOGO" device="XS"/>
+<part name="J3" library="Ai_Connectors" deviceset="1X04" device="" value="1X04"/>
+<part name="J1" library="Ai_Connectors" deviceset="1X04" device="NOFIRST" value="1X04NOFIRST"/>
 </parts>
 <sheets>
@@
 <instance part="GND1" gate="GND" x="99.06" y="86.36"/>
 <instance part="U$1" gate="G$1" x="91.44" y="114.3"/>
-<instance part="J1" gate="G$1" x="107.95" y="147.32"/>
-<instance part="J2" gate="G$1" x="147.32" y="147.32" rot="MR0"/>
 <instance part="GND2" gate="GND" x="148.59" y="86.36"/>
 <instance part="VDDIO2" gate="G$1" x="111.76" y="120.65"/>
-<instance part="JS1" gate="1" x="156.21" y="121.92" rot="R90"/>
-<instance part="JS2" gate="1" x="149.86" y="116.84" rot="R90"/>
-<instance part="JS3" gate="1" x="105.41" y="116.84" rot="R180"/>
+<instance part="PULL-UPS" gate="1" x="156.21" y="121.92" rot="R90"/>
+<instance part="MODE" gate="1" x="149.86" y="116.84" rot="R90"/>
+<instance part="VDDIO" gate="1" x="105.41" y="116.84" rot="R180"/>
 <instance part="U$2" gate="G$1" x="135.89" y="12.7"/>
+<instance part="J3" gate="G$1" x="147.32" y="144.78" rot="R180"/>
+<instance part="J1" gate="G$1" x="107.95" y="144.78" rot="MR180"/>
 </instances>
 <busses>
@@
 <net name="GND" class="0">
 <segment>
-<pinref part="J1" gate="G$1" pin="2"/>
 <wire x1="113.03" y1="144.78" x2="116.84" y2="144.78" width="0.1524" layer="91"/>
 <label x="116.84" y="144.78" size="1.27" layer="95" font="vector" ratio="10" xref="yes"/>
+<pinref part="J1" gate="G$1" pin="3"/>
 </segment>
 <segment>
@@
 </segment>
 <segment>
-<pinref part="J2" gate="G$1" pin="4"/>
 <wire x1="142.24" y1="149.86" x2="138.43" y2="149.86" width="0.1524" layer="91"/>
 <label x="138.43" y="149.86" size="1.27" layer="95" font="vector" ratio="10" rot="R180" xref="yes"/>
+<pinref part="J3" gate="G$1" pin="1"/>
 </segment>
 </net>
@@
 </segment>
 <segment>
-<pinref part="J1" gate="G$1" pin="1"/>
 <wire x1="113.03" y1="142.24" x2="116.84" y2="142.24" width="0.1524" layer="91"/>
 <label x="116.84" y="142.24" size="1.27" layer="95" font="vector" ratio="10" xref="yes"/>
+<pinref part="J1" gate="G$1" pin="4"/>
 </segment>
 <segment>
@@
 <wire x1="110.49" y1="116.84" x2="111.76" y2="116.84" width="0.1524" layer="91"/>
 <junction x="111.76" y="116.84"/>
-<pinref part="JS3" gate="1" pin="1"/>
+<pinref part="VDDIO" gate="1" pin="1"/>
 </segment>
 </net>
@@
 </segment>
 <segment>
-<pinref part="J2" gate="G$1" pin="2"/>
 <wire x1="142.24" y1="144.78" x2="138.43" y2="144.78" width="0.1524" layer="91"/>
 <label x="138.43" y="144.78" size="1.27" layer="95" font="vector" ratio="10" rot="R180" xref="yes"/>
+<pinref part="J3" gate="G$1" pin="3"/>
 </segment>
 </net>
@@
 </segment>
 <segment>
-<pinref part="J2" gate="G$1" pin="1"/>
 <wire x1="142.24" y1="142.24" x2="138.43" y2="142.24" width="0.1524" layer="91"/>
 <label x="138.43" y="142.24" size="1.27" layer="95" font="vector" ratio="10" rot="R180" xref="yes"/>
+<pinref part="J3" gate="G$1" pin="4"/>
 </segment>
 </net>
@@
 </segment>
 <segment>
-<pinref part="J1" gate="G$1" pin="4"/>
 <wire x1="113.03" y1="149.86" x2="116.84" y2="149.86" width="0.1524" layer="91"/>
 <label x="116.84" y="149.86" size="1.27" layer="95" font="vector" ratio="10" xref="yes"/>
+<pinref part="J1" gate="G$1" pin="1"/>
 </segment>
 </net>
@@
 <wire x1="99.06" y1="110.49" x2="87.63" y2="110.49" width="0.1524" layer="91"/>
 <label x="87.63" y="110.49" size="1.27" layer="95" font="vector" ratio="10" rot="R180" xref="yes"/>
-<pinref part="JS3" gate="1" pin="2"/>
+<pinref part="VDDIO" gate="1" pin="2"/>
 </segment>
 <segment>
-<pinref part="J1" gate="G$1" pin="3"/>
 <wire x1="113.03" y1="147.32" x2="116.84" y2="147.32" width="0.1524" layer="91"/>
 <label x="116.84" y="147.32" size="1.27" layer="95" font="vector" ratio="10" xref="yes"/>
+<pinref part="J1" gate="G$1" pin="2"/>
 </segment>
 <segment>
@@
 <label x="153.67" y="130.81" size="1.27" layer="95" font="vector" ratio="10" rot="R180" xref="yes"/>
 <wire x1="153.67" y1="128.27" x2="156.21" y2="128.27" width="0.1524" layer="91"/>
-<pinref part="JS1" gate="1" pin="2"/>
+<pinref part="PULL-UPS" gate="1" pin="2"/>
 <wire x1="156.21" y1="127" x2="156.21" y2="128.27" width="0.1524" layer="91"/>
-<pinref part="JS2" gate="1" pin="2"/>
+<pinref part="MODE" gate="1" pin="2"/>
 </segment>
 </net>
 <net name="CSB" class="0">
 <segment>
-<pinref part="J2" gate="G$1" pin="3"/>
 <wire x1="142.24" y1="147.32" x2="138.43" y2="147.32" width="0.1524" layer="91"/>
 <label x="138.43" y="147.32" size="1.27" layer="95" font="vector" ratio="10" rot="R180" xref="yes"/>
+<pinref part="J3" gate="G$1" pin="2"/>
 </segment>
 <segment>
@@
 <wire x1="144.78" y1="105.41" x2="149.86" y2="105.41" width="0.1524" layer="91"/>
 <wire x1="149.86" y1="105.41" x2="149.86" y2="111.76" width="0.1524" layer="91"/>
-<pinref part="JS2" gate="1" pin="1"/>
+<pinref part="MODE" gate="1" pin="1"/>
 <label x="144.78" y="105.918" size="1.27" layer="95" font="vector" ratio="10"/>
 </segment>
@@
 <wire x1="157.48" y1="115.57" x2="157.48" y2="113.03" width="0.1524" layer="91"/>
 <wire x1="153.67" y1="115.57" x2="156.21" y2="115.57" width="0.1524" layer="91"/>
-<pinref part="JS1" gate="1" pin="1"/>
+<pinref part="PULL-UPS" gate="1" pin="1"/>
 <wire x1="156.21" y1="115.57" x2="157.48" y2="115.57" width="0.1524" layer="91"/>
 <wire x1="156.21" y1="115.57" x2="156.21" y2="116.84" width="0.1524" layer="91"/>
